Commit message: update ros2_control

File: install/ros2-hoverboard-driver/share/ros2-hoverboard-driver/xacro/robot.urdf.xacro (robot description, xacro)
@@ -1,140 +1 @@
-<?xml version="1.0"?>
-<robot name="robot_mecatronica" xmlns:xacro="http://ros.org/wiki/xacro">
-  <!-- Include Colors Materials -->
-  <material name="red">
-    <color rgba="1 0 0 1"/> <!-- Rojo (RGB), opacidad 1 -->
-  </material>
-  <material name="black">
-    <color rgba="0 0 0 1"/> <!-- Negro -->
-  </material>
-  <material name="blue">
-    <color rgba="0 0 1 1"/> <!-- Azul -->
-  </material>
-  <!-- Include Robot Description -->
-  <link name="base_footprint"/>
-  <link name="base_link">
-    <visual>
-      <origin xyz="0 0 0" rpy="0 0 0" />
-      <geometry>
-        <box size="0.4 0.35 0.35"/> <!-- Dimensiones del chasis -->
-      </geometry>
-      <material name="red"/>
-    </visual>
-    <collision>
-      <origin xyz="0 0 0" rpy="0 0 0" />
-      <geometry>
-        <box size="0.4 0.35 0.35"/>
-      </geometry>
-    </collision>
-  </link>
-  <joint name="base_joint" type="fixed">
-    <parent link="base_footprint"/>
-    <child link="base_link" />
-    <origin xyz="0 0 0.08" rpy="0 0 0"/>
-  </joint>
-  <link name="right_wheel">
-    <visual>
-      <origin xyz="0 0 0" rpy="1.57 0 0" />
-      <geometry>
-        <cylinder length="0.05" radius="0.0825"/> <!-- Dimensiones de la rueda -->
-      </geometry>
-      <material name="black"/>
-    </visual>
-    <collision>
-    <origin xyz="-0.15 -0.16 -0.18" rpy="0 0 0"/> <!-- Ajusta estos valores -->
-      <geometry>
-        <cylinder length="0.05" radius="0.0825"/>
-      </geometry>
-    </collision>
-  </link>
-  <joint name="right_wheel" type="continuous">
-    <parent link="base_link"/>
-    <child link="right_wheel"/>
-    <origin xyz="-0.15 0.16 -0.18" rpy="0 0 0"/> <!-- Ajusta estos valores -->
-    <axis xyz="0 1 0"/>
-  </joint>
-  <link name="left_wheel">
-    <visual>
-      <origin xyz="0 0 0" rpy="-1.57 0 0" />
-      <geometry>
-        <cylinder length="0.05" radius="0.0825"/> <!-- Dimensiones de la rueda -->
-      </geometry>
-      <material name="black"/>
-    </visual>
-    <collision>
-      <origin xyz="0 0.015 0" rpy="-1.57 0 0" />
-      <geometry>
-        <cylinder length="0.05" radius="0.0825"/>
-      </geometry>
-    </collision>
-  </link>
-  <joint name="left_wheel" type="continuous">
-    <parent link="base_link"/>
-    <child link="left_wheel"/>
-    <origin xyz="-0.15 -0.16 -0.18" rpy="0 0 0"/> <!-- Ajusta estos valores -->
-    <axis xyz="0 1 0"/>
-  </joint>
-  <!-- Lidar -->
- <link name="laser">
-  <visual>
-    <origin xyz="0 0 0" rpy="0 0 0"/>
-    <geometry>
-      <cylinder length="0.05" radius="0.04"/>
-    </geometry>
-    <material name="blue"/>
-  </visual>
-  <collision>
-    <origin xyz="0 0 0" rpy="0 0 0"/>
-    <geometry>
-      <cylinder length="0.05" radius="0.04"/>
-    </geometry>
-  </collision>
-</link>
-<joint name="laser_joint" type="fixed">
-  <parent link="base_link"/>
-  <child link="laser"/>
-  <origin xyz="0.2 0 0.175" rpy="0 0 0"/>
-</joint>
-  <!-- Rueda guía izquierda -->
-<link name="front_left_guide_wheel">
-  <visual>
-    <origin xyz="0 0 0" rpy="-1.57 0 0"/> <!-- Ajusta la posición -->
-    <geometry>
-      <cylinder length="0.02" radius="0.025"/> <!-- Dimensiones de la rueda -->
-    </geometry>
-    <material name="black"/>
-  </visual>
-  <collision>
-    <origin xyz="0 0 0" rpy="0 0 0"/>
-    <geometry>
-      <cylinder length="0.02" radius="0.025"/>
-    </geometry>
-  </collision>
-</link>
-<joint name="front_left_guide_wheel_joint" type="fixed">
-  <parent link="base_link"/>
-  <child link="front_left_guide_wheel"/>
-  <origin xyz="0.15 -0.075 -0.18" rpy="0 0 0"/>
-</joint>
-<!-- Rueda guía derecha -->
-<link name="front_right_guide_wheel">
-  <visual>
-    <origin xyz="0 0 0" rpy="-1.57 0 0"/> <!-- Ajusta la posición -->
-    <geometry>
-      <cylinder length="0.02" radius="0.025"/> <!-- Dimensiones de la rueda -->
-    </geometry>
-    <material name="black"/>
-  </visual>
-  <collision>
-    <origin xyz="0 0 0" rpy="0 0 0"/>
-    <geometry>
-      <cylinder length="0.02" radius="0.025"/>
-    </geometry>
-  </collision>
-</link>
-<joint name="front_right_guide_wheel_joint" type="fixed">
-  <parent link="base_link"/>
-  <child link="front_right_guide_wheel"/>
-  <origin xyz="0.15 0.075 -0.18" rpy="0 0 0"/>
-</joint>
-</robot>
+/home/ros/Mapbot/src/ros2-hoverboard-driver/xacro/robot.urdf.xacro
